Commit message: adding gazebo files and the models they run

File: src/tfr_description/xacro/arm_model_overview.xacro (robot description, xacro)
@@ -1,11 +1,12 @@
 <?xml version="1.0"?>
+<!-- This file contains a top level description for the model of just
+    the arm without the Robot base -->
 <robot name="excavator" xmlns:xacro="http://www.ros.org/wiki/xacro">
   <!-- Top-level robot description -->
   <xacro:include filename="model_constants.xacro"/>
-  <xacro:include filename="model_base.xacro"/>
-  <xacro:include filename="model_arm.xacro"/>
+  <xacro:include filename="arm_without_base.xacro"/>
   <gazebo>
     <plugin name="gazebo_ros_control" filename="libgazebo_ros_control.so">
-      <robotNamespace>/</robotNamespace>
+      <robotNamespace>/tfr_arm</robotNamespace>
       <robotSimType>gazebo_ros_control/DefaultRobotHWSim</robotSimType>
     </plugin>

File: src/tfr_description/xacro/arm_without_base.xacro (robot description, xacro)
@@ -1,4 +1,17 @@
 <?xml version="1.0"?>
+<!-- Model of the arm without the joint that would atatch it to the base.
+    used for simulation the arm without the base -->
 <robot xmlns:xacro="http://www.ros.org/wiki/xacro" name="excavator">
+  <!-- attatch robot to world frame -->
+  <link name="world">
+    <!--<inertial>
+      <mass value="${100.0}" />
+      <inertia ixx="100.0" ixy="0.0" ixz="0.0" iyy="100.0" iyz="0.0" izz="100.0"/>
+    </inertial>-->
+  </link>
+  <joint name="fixed" type="fixed">
+    <parent link="world"/>
+    <child link="turntable"/>
+  </joint>
   <!--DIGGING ARM-->
   <link name="turntable">
@@ -24,5 +37,6 @@
     </inertial>
   </link>
-  <joint name="turntable_joint" type="revolute">
+  <!--Removed joint because for my simulation I am not including the base-->
+  <!--<joint name="turntable_joint" type="revolute">
     <parent link="base_link" />
     <child link="turntable" />
@@ -43,5 +57,5 @@
       <motorTorqueConstant>1</motorTorqueConstant>
     </actuator>
-  </transmission>
+  </transmission>-->
   <link name="lower_arm">
     <visual>

File: src/tfr_description/xacro/model_base.xacro (robot description, xacro)
@@ -1,4 +1,10 @@
 <?xml version="1.0"?>
 <robot xmlns:xacro="http://www.ros.org/wiki/xacro" name="excavator">
+  <!-- attatch robot to world frame-->
+  <link name="world"/>
+  <joint name="fixed" type="fixed">
+    <parent link="world"/>
+    <child link="base_link"/>
+  </joint>
   <!-- CHASSIS -->
   <link name="base_link" >
@@ -55,4 +61,9 @@
       <origin xyz="${tube_width / 2 - base_length / 2} 0 0" />
     </collision>
+    <!-- test -->
+    <inertial>
+      <mass value="1.0" />
+      <inertia ixx="1.0" ixy="0.0" ixz="0.0" iyy="1.0" iyz="0.0" izz="1.0"/>
+    </inertial>
   </link>
   <!-- DRIVEBASE -->
@@ -69,4 +80,9 @@
       </geometry>
     </collision>
+    <!-- test -->
+    <inertial>
+      <mass value="1.0" />
+      <inertia ixx="1.0" ixy="0.0" ixz="0.0" iyy="1.0" iyz="0.0" izz="1.0"/>
+    </inertial>
   </link>
   <joint name="left_tread_joint" type="fixed">
@@ -86,4 +102,9 @@
       </geometry>
     </collision>
+    <!-- test -->
+    <inertial>
+      <mass value="1.0" />
+      <inertia ixx="1.0" ixy="0.0" ixz="0.0" iyy="1.0" iyz="0.0" izz="1.0"/>
+    </inertial>
   </link>
   <joint name="right_tread_joint" type="fixed">
@@ -105,4 +126,9 @@
       <origin rpy="${pi/2} 0.0 0.0" />
     </collision>
+    <!-- test -->
+    <inertial>
+      <mass value="1.0" />
+      <inertia ixx="1.0" ixy="0.0" ixz="0.0" iyy="1.0" iyz="0.0" izz="1.0"/>
+    </inertial>
   </link>
   <joint name="tread_left_front_joint" type="fixed">
@@ -124,4 +150,9 @@
       <origin rpy="${pi/2} 0.0 0.0" />
     </collision>
+    <!-- test -->
+    <inertial>
+      <mass value="1.0" />
+      <inertia ixx="1.0" ixy="0.0" ixz="0.0" iyy="1.0" iyz="0.0" izz="1.0"/>
+    </inertial>
   </link>
   <joint name="tread_left_rear_joint" type="fixed">
@@ -143,4 +174,9 @@
       <origin rpy="${pi/2} 0.0 0.0" />
     </collision>
+    <!-- test -->
+    <inertial>
+      <mass value="1.0" />
+      <inertia ixx="1.0" ixy="0.0" ixz="0.0" iyy="1.0" iyz="0.0" izz="1.0"/>
+    </inertial>
   </link>
   <joint name="tread_right_front_joint" type="fixed">
@@ -162,4 +198,9 @@
       <origin rpy="${pi/2} 0.0 0.0" />
     </collision>
+    <!-- test -->
+    <inertial>
+      <mass value="1.0" />
+      <inertia ixx="1.0" ixy="0.0" ixz="0.0" iyy="1.0" iyz="0.0" izz="1.0"/>
+    </inertial>
   </link>
   <joint name="tread_right_rear_joint" type="fixed">
@@ -181,4 +222,9 @@
       <origin xyz="${tread_slope_length/2} 0.0 ${-1.25/2*itom}" />
     </collision>
+    <!-- test -->
+    <inertial>
+      <mass value="1.0" />
+      <inertia ixx="1.0" ixy="0.0" ixz="0.0" iyy="1.0" iyz="0.0" izz="1.0"/>
+    </inertial>
   </link>
   <joint name="front_right_slope_joint" type="fixed">
@@ -200,4 +246,9 @@
       <origin xyz="${tread_slope_length/2} 0.0 ${-1.25/2*itom}" />
     </collision>
+    <!-- test -->
+    <inertial>
+      <mass value="1.0" />
+      <inertia ixx="1.0" ixy="0.0" ixz="0.0" iyy="1.0" iyz="0.0" izz="1.0"/>
+    </inertial>
   </link>
   <joint name="front_left_slope_joint" type="fixed">
@@ -220,4 +271,9 @@
       <origin xyz="${bin_length} 0 ${-bin_height/2 + bin_height - (9.88 * itom) + (0.5*itom)}" />
     </collision>
+    <!-- test -->
+    <inertial>
+      <mass value="1.0" />
+      <inertia ixx="1.0" ixy="0.0" ixz="0.0" iyy="1.0" iyz="0.0" izz="1.0"/>
+    </inertial>
   </link>
   <joint name="bin_joint" type="revolute">
@@ -239,4 +295,9 @@
       </geometry>
     </collision>
+    <!-- test -->
+    <inertial>
+      <mass value="1.0" />
+      <inertia ixx="1.0" ixy="0.0" ixz="0.0" iyy="1.0" iyz="0.0" izz="1.0"/>
+    </inertial>
   </link>
   <joint name="bin_right_joint" type="fixed">
@@ -256,4 +317,9 @@
       </geometry>
     </collision>
+    <!-- test -->
+    <inertial>
+      <mass value="1.0" />
+      <inertia ixx="1.0" ixy="0.0" ixz="0.0" iyy="1.0" iyz="0.0" izz="1.0"/>
+    </inertial>
   </link>
   <joint name="bin_left_joint" type="fixed">
@@ -273,4 +339,9 @@
       </geometry>
     </collision>
+    <!-- test -->
+    <inertial>
+      <mass value="1.0" />
+      <inertia ixx="1.0" ixy="0.0" ixz="0.0" iyy="1.0" iyz="0.0" izz="1.0"/>
+    </inertial>
   </link>
   <joint name="bin_bottom_joint" type="fixed">
@@ -292,4 +363,9 @@
       <origin xyz="0 0 ${-bin_height*sqrt2*0.5}"/>
     </collision>
+    <!-- test -->
+    <inertial>
+      <mass value="1.0" />
+      <inertia ixx="1.0" ixy="0.0" ixz="0.0" iyy="1.0" iyz="0.0" izz="1.0"/>
+    </inertial>
   </link>
   <joint name="bin_slope_joint" type="fixed">
@@ -311,4 +387,9 @@
       <origin xyz=" ${bin_back_offset}  0 0"/>
     </collision>
+    <!-- test -->
+    <inertial>
+      <mass value="1.0" />
+      <inertia ixx="1.0" ixy="0.0" ixz="0.0" iyy="1.0" iyz="0.0" izz="1.0"/>
+    </inertial>
   </link>
   <joint name="bin_slope_2_joint" type="fixed">

File: src/tfr_description/xacro/model_constants.xacro (robot description, xacro)
@@ -9,4 +9,5 @@
   <xacro:property name="sqrt2" value="1.41421" />
   <!-- Drivebase parameters -->
+  <xacro:property name="base_mass" value="${25.0}"/>
   <xacro:property name="base_length" value="${50*itom}" />
   <xacro:property name="tube_width" value="${2*itom}" />
@@ -15,4 +16,6 @@
   <xacro:property name="drivebase_total_height" value="${6*itom}" />
   <!-- Drivetrain parameters -->
+  <xacro:property name="tred_left_mass" value="${30.0}" />
+  <xacro:property name="tred_right_mass" value="${30.0}" />
   <xacro:property name="tread_end_radius" value="${(15.5/2)*itom}" />
   <xacro:property name="tread_mid_height" value="${19*itom}" />
@@ -25,4 +28,5 @@
   <!-- Length of top of bin, length of bottom is 13.86 -->
   <!-- Using the bigger size as a box instead of making complex angled shape -->
+  <xacro:property name="bin_mass" value="${10.0}" />
   <xacro:property name="bin_length" value="${36*itom}" />
   <xacro:property name="bin_width" value="${13.5*itom}" />
@@ -31,4 +35,5 @@
   <xacro:property name="bin_back_offset" value="${6.5*itom}" />
   <!-- Turntable parameters -->
+  <xacro:property name="turntable_mass" value="${25.0}"/>
   <xacro:property name="turntable_radius" value="${4.92*itom}" />
   <!-- 1" in model plus undefined height for mounting and extra components -->
@@ -36,21 +41,24 @@
   <xacro:property name="turntable_height" value="${2.25*itom}" />
   <!-- Lower arm parameters -->
+  <xacro:property name="lower_arm_mass" value="${28.0}"/>
   <xacro:property name="lower_arm_length" value="${22*itom}" />
   <xacro:property name="lower_arm_primary_length" value="${16*itom}" />
   <xacro:property name="lower_arm_width" value="${6*itom}" />
   <xacro:property name="lower_arm_height" value="${6*itom}" />
-  <xacro:property name="lower_arm_min" value="0.1092" />
-  <xacro:property name="lower_arm_max" value="1.395" />
+  <xacro:property name="lower_arm_min" value="0.104" />
+  <xacro:property name="lower_arm_max" value="1.55" />
   <!-- Upper arm parameters -->
+  <xacro:property name="upper_arm_mass" value="${10.0}"/>
   <xacro:property name="upper_arm_length" value="${20*itom}" />
   <xacro:property name="upper_arm_width" value="${4.75*itom}" />
   <xacro:property name="upper_arm_height" value="${5*itom}" />
-  <xacro:property name="upper_arm_min" value="1.029"/>
-  <xacro:property name="upper_arm_max" value="2.28"/>
+  <xacro:property name="upper_arm_min" value="0.98"/>
+  <xacro:property name="upper_arm_max" value="2.4"/>
   <!-- Scoop parameters -->
+  <xacro:property name="scoop_mass" value="${5.0}"/>
   <xacro:property name="scoop_width" value="${8.5*itom}" />
   <xacro:property name="scoop_length" value="${12*itom}" />
   <xacro:property name="scoop_diameter" value="${12.5*itom}" />
-  <xacro:property name="scoop_min" value="-1.235" />
-  <xacro:property name="scoop_max" value="1.539" />
+  <xacro:property name="scoop_min" value="-1.16614" />
+  <xacro:property name="scoop_max" value="1.62" />
 </robot>
