Commit message: corrected arm model controller

File: src/tfr_description/xacro/arm_without_base.xacro (robot description, xacro)
@@ -4,10 +4,5 @@
 <robot xmlns:xacro="http://www.ros.org/wiki/xacro" name="excavator">
   <!-- attatch robot to world frame -->
-  <link name="world">
-    <!--<inertial>
-      <mass value="${100.0}" />
-      <inertia ixx="100.0" ixy="0.0" ixz="0.0" iyy="100.0" iyz="0.0" izz="100.0"/>
-    </inertial>-->
-  </link>
+  <link name="world"/>
   <joint name="fixed" type="fixed">
     <parent link="world"/>
@@ -30,32 +25,11 @@
     <!-- test -->
     <inertial>
-      <mass value="20.0" />
-      <!--<inertia ixx="${0.0833333 * turntable_mass * (3.0 * turntable_radius * turntable_radius + turntable_height * turntable_height)}" ixy="0.0" ixz="0.0"
+      <mass value="${turntable_mass}" />
+      <inertia ixx="${0.0833333 * turntable_mass * (3.0 * turntable_radius * turntable_radius + turntable_height * turntable_height)}" ixy="0.0" ixz="0.0"
         iyy="${0.0833333 * turntable_mass * (3.0 * turntable_radius * turntable_radius + turntable_height * turntable_height)}" iyz="0.0"
-        izz="${0.5 * turntable_mass * turntable_radius * turntable_radius}" />-->
-      <inertia ixx="20.0" ixy="0.0" ixz="0.0" iyy="20.0" iyz="0.0" izz="20.0"/>
-    </inertial>
-  </link>
-  <!--Removed joint because for my simulation I am not including the base-->
-  <!--<joint name="turntable_joint" type="revolute">
-    <parent link="base_link" />
-    <child link="turntable" />
-    <origin xyz="${base_length/2-turntable_radius} 0 ${drivebase_front_beam_height/2}" rpy="0 0 ${pi}" />
-    <axis xyz="0 0 1" />
-    <limit effort="1.0" velocity="1.0" lower="${-1.1*pi}" upper="${1.1*pi}" />
-  </joint>
-  <transmission name="turntable_tran">
-    <type>transmission_interface/SimpleTransmission</type>
-    <joint name="turntable_joint">
-      <hardwareInterface>hardware_interface/EffortJointInterface
-      </hardwareInterface>
-    </joint>
-    <actuator name="turntable_motor">
-      <hardwareInterface>hardware_interface/EffortJointInterface
-      </hardwareInterface>
-      <mechanicalReduction>1</mechanicalReduction>
-      <motorTorqueConstant>1</motorTorqueConstant>
-    </actuator>
-  </transmission>-->
+        izz="${0.5 * turntable_mass * turntable_radius * turntable_radius}" />
+      <!--<inertia ixx="20.0" ixy="0.0" ixz="0.0" iyy="20.0" iyz="0.0" izz="20.0"/>-->
+    </inertial>
+  </link>
   <link name="lower_arm">
     <visual>
@@ -73,9 +47,9 @@
     <!-- test -->
     <inertial>
-      <mass value="15.0" />
-      <!--<inertia ixx="${0.0833333 * lower_arm_mass * (lower_arm_width*lower_arm_width + lower_arm_primary_length*lower_arm_primary_length)}" ixy="0.0" ixz="0.0"
+      <mass value="${lower_arm_mass}" />
+      <inertia ixx="${0.0833333 * lower_arm_mass * (lower_arm_width*lower_arm_width + lower_arm_primary_length*lower_arm_primary_length)}" ixy="0.0" ixz="0.0"
         iyy="${0.0833333 * lower_arm_mass * (lower_arm_height*lower_arm_height + lower_arm_primary_length*lower_arm_primary_length)}" iyz="0.0"
-        izz="${0.0833333 * lower_arm_mass * (lower_arm_height*lower_arm_height + lower_arm_width*lower_arm_width)}" />-->
-      <inertia ixx="15.0" ixy="0.0" ixz="0.0" iyy="15.0" iyz="0.0" izz="15.0"/>
+        izz="${0.0833333 * lower_arm_mass * (lower_arm_height*lower_arm_height + lower_arm_width*lower_arm_width)}" />
+      <!--<inertia ixx="15.0" ixy="0.0" ixz="0.0" iyy="15.0" iyz="0.0" izz="15.0"/>-->
     </inertial>
   </link>
@@ -91,13 +65,9 @@
     <type>transmission_interface/SimpleTransmission</type>
     <joint name="lower_arm_joint">
-      <!--<hardwareInterface>hardware_interface/EffortJointInterface
-      </hardwareInterface>-->
-      <hardwareInterface>hardware_interface/PositionJointInterface
+      <hardwareInterface>hardware_interface/EffortJointInterface
       </hardwareInterface>
     </joint>
     <actuator name="lower_motor">
-      <!--<hardwareInterface>hardware_interface/EffortJointInterface
-      </hardwareInterface>-->
-      <hardwareInterface>hardware_interface/PositionJointInterface
+      <hardwareInterface>hardware_interface/EffortJointInterface
       </hardwareInterface>
       <mechanicalReduction>1</mechanicalReduction>
@@ -118,7 +88,6 @@
     <!-- test -->
     <inertial>
-      <mass value="15.0" />
-      <!--<inertia ixx="0.0833333 * lower_arm_mass" ixy="0.0" ixz="0.0" iyy="0.0833333 * lower_arm_mass" iyz="0.0" izz="0.0833333 * lower_arm_mass"/> -->
-      <inertia ixx="15.0" ixy="0.0" ixz="0.0" iyy="15.0" iyz="0.0" izz="15.0"/>
+      <mass value="2.3" />
+      <inertia ixx="${0.0833333 * 2.3}" ixy="0.0" ixz="0.0" iyy="${0.0833333 * 2.3}" iyz="0.0" izz="${0.0833333 * 2.3}"/>
     </inertial>
   </link>
@@ -143,7 +112,6 @@
     <!-- test -->
     <inertial>
-      <mass value="15.0" />
-      <!--<inertia ixx="0.0833333 * lower_arm_mass" ixy="0.0" ixz="0.0" iyy="0.0833333 * lower_arm_mass" iyz="0.0" izz="0.0833333 * lower_arm_mass"/>  -->
-      <inertia ixx="15.0" ixy="0.0" ixz="0.0" iyy="15.0" iyz="0.0" izz="15.0"/>
+      <mass value="2.3" />
+      <inertia ixx="${0.0833333 * 2.3}" ixy="0.0" ixz="0.0" iyy="${0.0833333 * 2.3}" iyz="0.0" izz="${0.0833333 * 2.3}"/>
     </inertial>
   </link>
@@ -168,9 +136,8 @@
     <!-- test -->
     <inertial>
-      <mass value="10.0" />
-      <!--<inertia ixx="${0.0833333 * upper_arm_mass * (upper_arm_width*upper_arm_width + upper_arm_length*upper_arm_length)}" ixy="0.0" ixz="0.0"
+      <mass value="${upper_arm_mass}" />
+      <inertia ixx="${0.0833333 * upper_arm_mass * (upper_arm_width*upper_arm_width + upper_arm_length*upper_arm_length)}" ixy="0.0" ixz="0.0"
         iyy="${0.0833333 * upper_arm_mass * (upper_arm_height*upper_arm_height + upper_arm_length*upper_arm_length)}" iyz="0.0"
-        izz="${0.0833333 * upper_arm_mass * (upper_arm_height*upper_arm_height + upper_arm_width*upper_arm_width)}" /> -->
-      <inertia ixx="10.0" ixy="0.0" ixz="0.0" iyy="10.0" iyz="0.0" izz="10.0"/>
+        izz="${0.0833333 * upper_arm_mass * (upper_arm_height*upper_arm_height + upper_arm_width*upper_arm_width)}" />
     </inertial>
   </link>
@@ -186,9 +153,9 @@
     <type>transmission_interface/SimpleTransmission</type>
     <joint name="upper_arm_joint">
-      <hardwareInterface>hardware_interface/PositionJointInterface
+      <hardwareInterface>hardware_interface/EffortJointInterface
       </hardwareInterface>
     </joint>
     <actuator name="upper_motor">
-      <hardwareInterface>hardware_interface/PositionJointInterface
+      <hardwareInterface>hardware_interface/EffortJointInterface
       </hardwareInterface>
       <mechanicalReduction>1</mechanicalReduction>
@@ -211,9 +178,8 @@
     <!-- test -->
     <inertial>
-      <mass value="5.0" />
-      <!--<inertia ixx="${0.0833333 * scoop_mass * (scoop_width*scoop_width + (scoop_diameter/2)*(scoop_diameter/2))}" ixy="0.0" ixz="0.0"
+      <mass value="${scoop_mass}" />
+      <inertia ixx="${0.0833333 * scoop_mass * (scoop_width*scoop_width + (scoop_diameter/2)*(scoop_diameter/2))}" ixy="0.0" ixz="0.0"
         iyy="${0.0833333 * scoop_mass * (scoop_length*scoop_length + (scoop_diameter/2)*(scoop_diameter/2))}" iyz="0.0"
-        izz="${0.0833333 * scoop_mass * (scoop_length*scoop_length + scoop_width*scoop_width)}" />-->
-      <inertia ixx="5.0" ixy="0.0" ixz="0.0" iyy="5.0" iyz="0.0" izz="5.0"/>
+        izz="${0.0833333 * scoop_mass * (scoop_length*scoop_length + scoop_width*scoop_width)}" />
     </inertial>
   </link>
@@ -229,9 +195,9 @@
     <type>transmission_interface/SimpleTransmission</type>
     <joint name="scoop_joint">
-      <hardwareInterface>hardware_interface/PositionJointInterface
+      <hardwareInterface>hardware_interface/EffortJointInterface
       </hardwareInterface>
     </joint>
     <actuator name="end_motor">
-      <hardwareInterface>hardware_interface/PositionJointInterface
+      <hardwareInterface>hardware_interface/EffortJointInterface
       </hardwareInterface>
       <mechanicalReduction>1</mechanicalReduction>

File: src/tfr_description/xacro/model_constants.xacro (robot description, xacro)
@@ -9,5 +9,4 @@
   <xacro:property name="sqrt2" value="1.41421" />
   <!-- Drivebase parameters -->
-  <xacro:property name="base_mass" value="${25.0}"/>
   <xacro:property name="base_length" value="${50*itom}" />
   <xacro:property name="tube_width" value="${2*itom}" />
@@ -16,6 +15,4 @@
   <xacro:property name="drivebase_total_height" value="${6*itom}" />
   <!-- Drivetrain parameters -->
-  <xacro:property name="tred_left_mass" value="${30.0}" />
-  <xacro:property name="tred_right_mass" value="${30.0}" />
   <xacro:property name="tread_end_radius" value="${(15.5/2)*itom}" />
   <xacro:property name="tread_mid_height" value="${19*itom}" />
@@ -28,5 +25,4 @@
   <!-- Length of top of bin, length of bottom is 13.86 -->
   <!-- Using the bigger size as a box instead of making complex angled shape -->
-  <xacro:property name="bin_mass" value="${10.0}" />
   <xacro:property name="bin_length" value="${36*itom}" />
   <xacro:property name="bin_width" value="${13.5*itom}" />
@@ -35,5 +31,5 @@
   <xacro:property name="bin_back_offset" value="${6.5*itom}" />
   <!-- Turntable parameters -->
-  <xacro:property name="turntable_mass" value="${25.0}"/>
+  <xacro:property name="turntable_mass" value="${16.0}"/>
   <xacro:property name="turntable_radius" value="${4.92*itom}" />
   <!-- 1" in model plus undefined height for mounting and extra components -->
@@ -41,5 +37,5 @@
   <xacro:property name="turntable_height" value="${2.25*itom}" />
   <!-- Lower arm parameters -->
-  <xacro:property name="lower_arm_mass" value="${28.0}"/>
+  <xacro:property name="lower_arm_mass" value="${8.2}"/>
   <xacro:property name="lower_arm_length" value="${22*itom}" />
   <xacro:property name="lower_arm_primary_length" value="${16*itom}" />
@@ -49,5 +45,5 @@
   <xacro:property name="lower_arm_max" value="1.55" />
   <!-- Upper arm parameters -->
-  <xacro:property name="upper_arm_mass" value="${10.0}"/>
+  <xacro:property name="upper_arm_mass" value="${6.4}"/>
   <xacro:property name="upper_arm_length" value="${20*itom}" />
   <xacro:property name="upper_arm_width" value="${4.75*itom}" />
@@ -56,5 +52,5 @@
   <xacro:property name="upper_arm_max" value="2.4"/>
   <!-- Scoop parameters -->
-  <xacro:property name="scoop_mass" value="${5.0}"/>
+  <xacro:property name="scoop_mass" value="${3.6}"/>
   <xacro:property name="scoop_width" value="${8.5*itom}" />
   <xacro:property name="scoop_length" value="${12*itom}" />

Commit message: some model tweaking and added more poses to tfr_gazebo_arm_moveit

File: src/tfr_description/xacro/arm_without_base.xacro (robot description, xacro)
@@ -88,5 +88,5 @@
     <!-- test -->
     <inertial>
-      <mass value="2.3" />
+      <mass value=".23" />
       <inertia ixx="${0.0833333 * 2.3}" ixy="0.0" ixz="0.0" iyy="${0.0833333 * 2.3}" iyz="0.0" izz="${0.0833333 * 2.3}"/>
     </inertial>
@@ -112,5 +112,5 @@
     <!-- test -->
     <inertial>
-      <mass value="2.3" />
+      <mass value=".23" />
       <inertia ixx="${0.0833333 * 2.3}" ixy="0.0" ixz="0.0" iyy="${0.0833333 * 2.3}" iyz="0.0" izz="${0.0833333 * 2.3}"/>
     </inertial>

File: src/tfr_description/xacro/model_constants.xacro (robot description, xacro)
@@ -31,5 +31,5 @@
   <xacro:property name="bin_back_offset" value="${6.5*itom}" />
   <!-- Turntable parameters -->
-  <xacro:property name="turntable_mass" value="${16.0}"/>
+  <xacro:property name="turntable_mass" value="${1.6}"/>
   <xacro:property name="turntable_radius" value="${4.92*itom}" />
   <!-- 1" in model plus undefined height for mounting and extra components -->
@@ -37,5 +37,5 @@
   <xacro:property name="turntable_height" value="${2.25*itom}" />
   <!-- Lower arm parameters -->
-  <xacro:property name="lower_arm_mass" value="${8.2}"/>
+  <xacro:property name="lower_arm_mass" value="${.82}"/>
   <xacro:property name="lower_arm_length" value="${22*itom}" />
   <xacro:property name="lower_arm_primary_length" value="${16*itom}" />
@@ -45,5 +45,5 @@
   <xacro:property name="lower_arm_max" value="1.55" />
   <!-- Upper arm parameters -->
-  <xacro:property name="upper_arm_mass" value="${6.4}"/>
+  <xacro:property name="upper_arm_mass" value="${.64}"/>
   <xacro:property name="upper_arm_length" value="${20*itom}" />
   <xacro:property name="upper_arm_width" value="${4.75*itom}" />
@@ -52,5 +52,5 @@
   <xacro:property name="upper_arm_max" value="2.4"/>
   <!-- Scoop parameters -->
-  <xacro:property name="scoop_mass" value="${3.6}"/>
+  <xacro:property name="scoop_mass" value="${.36}"/>
   <xacro:property name="scoop_width" value="${8.5*itom}" />
   <xacro:property name="scoop_length" value="${12*itom}" />
