Commit message: Modify drivebase model to no longer link base_link to a world frame in order to resolve conflict with transform from base_footprint. Add fake odometry node inorder to initialize odometry which in turn allows the nav stack to begin mapping. Add launch file to display obstacles found by realsense.

File: src/tfr_description/xacro/model_base.xacro (robot description, xacro)
@@ -1,10 +1,4 @@
 <?xml version="1.0"?>
 <robot xmlns:xacro="http://www.ros.org/wiki/xacro" name="excavator">
-  <!-- attatch robot to world frame-->
-  <link name="world"/>
-  <joint name="fixed" type="fixed">
-    <parent link="world"/>
-    <child link="base_link"/>
-  </joint>
   <!-- CHASSIS -->
   <link name="base_link" >

Commit message: Added rplidar and Cartographer packages to src, and modified launch files to call rplidar. Also modified the model to include rplidar joint.

File: src/tfr_description/xacro/model_base.xacro (robot description, xacro)
@@ -61,4 +61,12 @@
     </inertial>
   </link>
+  <!-- Not final orientation or name, only for testing -->
+  <!-- RPLidar 2D LIDAR -->
+  <xacro:macro name="sensor_rplidar" params="parent">
+      <joint name="laser" type="fixed">
+          <origin xyz="${(tube_width / 2 - base_length / 2)/2} 0 ${tube_width + 0.1}" rpy="0 0 0" />
+          <parent link="base_link" />
+      </joint>
+  </xacro:macro>
   <!-- DRIVEBASE -->
   <!-- A general tread huge block: may be refined later for slightly better operational motion -->

Commit message: added a base footprint to the model

File: src/tfr_description/xacro/model_base.xacro (robot description, xacro)
@@ -1,4 +1,11 @@
 <?xml version="1.0"?>
 <robot xmlns:xacro="http://www.ros.org/wiki/xacro" name="excavator">
+  <!--world links -->
+  <link name="base_footprint" />
+  <joint name="base_footprint_joint" type="fixed">
+    <origin xyz="0 0 0.017" rpy="0 0 0" />
+    <parent link="base_footprint" />
+    <child link="base_link" />
+  </joint>
   <!-- CHASSIS -->
   <link name="base_link" >
